File: TurnSignal.kicad_pcb (KiCad board)
At the start: 2 copper layers, 61.4 x 19.6 mm, 23 parts, among them J1 B2B-PH-K-S_LF__SN_, J2 Conn_01x05_Pin, J5 Conn_01x03_Pin, J6 Conn_01x03_Pin, Q1 FMMT491A, Q2 FMMT491A, U1 LM555xM

Commit message: idk
Parts:
- removed the G*** at (115.0, 128.8)
- added ?: , , F.Cu at (119.3, 95.9)
- added ?: , , F.Cu at (142.8, 95.9)
- added ?: , , F.Cu at (150.1, 95.9)
- added ?: , , F.Cu at (112.0, 95.9)
- moved J1 0.32 mm to (135.8, 97.2)
Routing:
- net GND: track 2.00 -> 6.07 mm
- net +9V: track 3.94 -> 7.28 mm

Commit message: d
Parts:
- added G***: LOGO, LOGO, B.Cu at (116.9, 121.2)
- moved G*** 45.8 mm to (126.6, 104.1)
- moved G*** 41.4 mm to (96.1, 83.1)

Commit message: :)
Parts:
- moved G*** 69.2 mm to (63.6, 132.6)
- moved G*** 25.4 mm to (92.1, 127.1)
- moved G*** 8.40 mm to (88.8, 87.1)
Other:
- board text removed: "+"
